Commit message: 2nd

File: src/articubot_one/description/gazebo_control.xacro (robot description, xacro)
@@ -2,26 +2,13 @@
 <robot xmlns:xacro="http://www.ros.org/wiki/xacro">
     <gazebo>
-        <plugin name='front' filename='libgazebo_ros_diff_drive.so'>
+        <plugin name='diff_drive' filename='libgazebo_ros_diff_drive.so'>
             <!-- Wheel Information -->
+            <num_wheel_pairs>2</num_wheel_pairs>
             <left_joint>front_left_wheel_joint</left_joint>
             <right_joint>front_right_wheel_joint</right_joint>
-            <wheel_separation>0.35</wheel_separation>  <!-- Distance between wheels (update if needed) -->
-            <wheel_diameter>0.1</wheel_diameter>        <!-- Diameter of the wheels (update if needed) -->
-            <!-- Limits -->
-            <max_wheel_torque>200</max_wheel_torque>
-            <max_wheel_acceleration>10.0</max_wheel_acceleration>
-            <!-- Output -->
-            <odometry_frame>odom</odometry_frame>
-            <robot_base_frame>base_link</robot_base_frame>
-            <publish_odom>true</publish_odom>
-            <publish_odom_tf>true</publish_odom_tf>
-            <publish_wheel_tf>true</publish_wheel_tf>
-        </plugin>
-        <plugin name='back' filename='libgazebo_ros_diff_drive.so'>
-            <!-- Wheel Information -->
             <left_joint>back_left_wheel_joint</left_joint>
             <right_joint>back_right_wheel_joint</right_joint>
-            <wheel_separation>0.35</wheel_separation>  <!-- Distance between wheels (update if needed) -->
-            <wheel_diameter>0.1</wheel_diameter>        <!-- Diameter of the wheels (update if needed) -->
+            <wheel_separation>0.35z</wheel_separation>
+            <wheel_diameter>0.14</wheel_diameter>
             <!-- Limits -->
             <max_wheel_torque>200</max_wheel_torque>

File: src/articubot_one/description/gripper.xacro (robot description, xacro)
@@ -4,5 +4,5 @@
     <link name="gripper_base">
         <visual>
-            <origin xyz="0 -0.3 0" rpy="0 0 0"/>
+            <origin xyz="0 0 0.05" rpy="0 0 0"/>
             <geometry>
                 <box size="0.35 0.05 0.05"/>
@@ -11,5 +11,5 @@
         </visual>
         <collision>
-            <origin xyz="0 -0.3 0" rpy="0 0 0"/>
+            <origin xyz="0 0 0.05" rpy="0 0 0"/>
             <geometry>
                 <box size="0.35 0.05 0.05"/>
@@ -35,5 +35,5 @@
         </collision>
         <xacro:inertial_box mass="0.5" x="0.35" y="0.05" z="0.05" >
-            <origin xyz="0 -0.3 0" rpy="0 0 0"/>
+            <origin xyz="0 0 0.05" rpy="0 0 0"/>
         </xacro:inertial_box>
     </link>
@@ -41,12 +41,12 @@
     <link name="gripper_finger_left">
         <visual>
-            <origin xyz="-0.075 -0.4 0" rpy="0 0 0"/>
+            <origin xyz="-0.075 -0.1 0.05" rpy="0 0 0"/>
             <geometry>
                 <box size="0.0225 0.2 0.05"/>
             </geometry>
-            <material name="gray"/>
+            <material name="orange"/>
         </visual>
         <collision>
-            <origin xyz="-0.075 -0.4 0" rpy="0 0 0"/>
+            <origin xyz="-0.075 -0.1 0.05" rpy="0 0 0"/>
             <geometry>
                 <box size="0.0225 0.2 0.1"/>
@@ -72,5 +72,5 @@
         </collision>
         <xacro:inertial_box mass="0.3" x="0.0225" y="0.2" z="0.05" >
-            <origin xyz="-0.075 -0.4 0" rpy="0 0 0"/>
+            <origin xyz="-0.075 -0.1 0.05" rpy="0 0 0"/>
         </xacro:inertial_box>
     </link>
@@ -78,12 +78,12 @@
     <link name="gripper_finger_right">
         <visual>
-            <origin xyz="0.075 -0.4 0" rpy="0 0 0"/>
+            <origin xyz="0.075 -0.10 0.05" rpy="0 0 0"/>
             <geometry>
                 <box size="0.0225 0.2 0.05"/>
             </geometry>
-            <material name="gray"/>
+            <material name="orange"/>
         </visual>
         <collision>
-            <origin xyz="0.075 -0.4 0" rpy="0 0 0"/>
+            <origin xyz="0.075 -0.10 0.05" rpy="0 0 0"/>
             <geometry>
                 <box size="0.0225 0.2 0.1"/>
@@ -109,5 +109,5 @@
         </collision>
         <xacro:inertial_box mass="0.3" x="0.0225" y="0.2" z="0.05" >
-            <origin xyz="0.075 -0.4 0" rpy="0 0 0"/>
+            <origin xyz="0.075 -0.10 0.05" rpy="0 0 0"/>
         </xacro:inertial_box>
     </link>
@@ -125,5 +125,5 @@
         <parent link="gripper_base"/>
         <child link="gripper_finger_left"/>
-        <origin xyz="-0.03 0 0" rpy="0 0 0"/>
+        <origin xyz="-0.075 0 0" rpy="0 0 0"/>
         <axis xyz="1 0 0"/>
         <limit effort="100" lower="0" upper="0.1" velocity="0.1"/>
@@ -133,5 +133,5 @@
         <parent link="gripper_base"/>
         <child link="gripper_finger_right"/>
-        <origin xyz="0.03 0 0" rpy="0 0 0"/>
+        <origin xyz="0.075 0 0" rpy="0 0 0"/>
         <axis xyz="1 0 0"/>
         <limit effort="100" lower="-0.1" upper="0" velocity="0.1"/>
@@ -148,5 +148,5 @@
     </gazebo>
     <gazebo reference="gripper_finger_left">
-        <material>Gazebo/Gray</material>
+        <material>Gazebo/Orange</material>
         <gravity>true</gravity>
         <ode>
@@ -160,5 +160,5 @@
     </gazebo>
     <gazebo reference="gripper_finger_right">
-        <material>Gazebo/Gray</material>
+        <material>Gazebo/Orange</material>
         <gravity>true</gravity>
         <ode>

File: src/articubot_one/description/robot_core.xacro (robot description, xacro)
@@ -73,5 +73,5 @@
                 <cylinder length="0.03" radius="0.07" />
             </geometry>
-            <material name="black"/>
+            <material name="blue"/>
         </visual>
         <collision>
@@ -85,5 +85,5 @@
     </link>
     <gazebo reference="front_left_wheel">
-        <material>Gazebo/Black</material>
+        <material>Gazebo/Blue</material>
     </gazebo>
     <link name="front_right_wheel">
@@ -92,5 +92,5 @@
                 <cylinder length="0.03" radius="0.07" />
             </geometry>
-            <material name="black"/>
+            <material name="red"/>
         </visual>
         <collision>
@@ -104,5 +104,5 @@
     </link>
     <gazebo reference="front_right_wheel">
-        <material>Gazebo/Black</material>
+        <material>Gazebo/Red</material>
     </gazebo>
     <link name="back_left_wheel">
@@ -111,5 +111,5 @@
                 <cylinder length="0.03" radius="0.07" />
             </geometry>
-            <material name="black"/>
+            <material name="orange"/>
         </visual>
         <collision>
@@ -123,5 +123,5 @@
     </link>
     <gazebo reference="back_left_wheel">
-        <material>Gazebo/Black</material>
+        <material>Gazebo/Orange</material>
     </gazebo>
     <link name="back_right_wheel">
@@ -130,5 +130,5 @@
                 <cylinder length="0.03" radius="0.07" />
             </geometry>
-            <material name="black"/>
+            <material name="green"/>
         </visual>
         <collision>
@@ -142,5 +142,5 @@
     </link>
     <gazebo reference="back_right_wheel">
-        <material>Gazebo/Black</material>
+        <material>Gazebo/Green</material>
     </gazebo>
     <!-- Wheel Joint -->
