Commit message: 3rd

File: src/articubot_one/description/gripper.xacro (robot description, xacro)
@@ -4,5 +4,5 @@
     <link name="gripper_base">
         <visual>
-            <origin xyz="0 0 0.05" rpy="0 0 0"/>
+            <origin xyz="0 0 0.025" rpy="0 0 0"/>
             <geometry>
                 <box size="0.35 0.05 0.05"/>
@@ -11,5 +11,5 @@
         </visual>
         <collision>
-            <origin xyz="0 0 0.05" rpy="0 0 0"/>
+            <origin xyz="0 0 0.025" rpy="0 0 0"/>
             <geometry>
                 <box size="0.35 0.05 0.05"/>
@@ -35,5 +35,5 @@
         </collision>
         <xacro:inertial_box mass="0.5" x="0.35" y="0.05" z="0.05" >
-            <origin xyz="0 0 0.05" rpy="0 0 0"/>
+            <origin xyz="0 0 0.025" rpy="0 0 0"/>
         </xacro:inertial_box>
     </link>
@@ -41,12 +41,12 @@
     <link name="gripper_finger_left">
         <visual>
-            <origin xyz="-0.075 -0.1 0.05" rpy="0 0 0"/>
+            <origin xyz="-0.025 -0.1 0.025" rpy="0 0 0"/>
             <geometry>
-                <box size="0.0225 0.2 0.05"/>
+                <box size="0.0225 0.2 0.025"/>
             </geometry>
-            <material name="orange"/>
+            <material name="black"/>
         </visual>
         <collision>
-            <origin xyz="-0.075 -0.1 0.05" rpy="0 0 0"/>
+            <origin xyz="-0.025 -0.1 0.025" rpy="0 0 0"/>
             <geometry>
                 <box size="0.0225 0.2 0.1"/>
@@ -72,5 +72,5 @@
         </collision>
         <xacro:inertial_box mass="0.3" x="0.0225" y="0.2" z="0.05" >
-            <origin xyz="-0.075 -0.1 0.05" rpy="0 0 0"/>
+            <origin xyz="-0.025 -0.1 0.025" rpy="0 0 0"/>
         </xacro:inertial_box>
     </link>
@@ -78,12 +78,12 @@
     <link name="gripper_finger_right">
         <visual>
-            <origin xyz="0.075 -0.10 0.05" rpy="0 0 0"/>
+            <origin xyz="0.025 -0.10 0.025" rpy="0 0 0"/>
             <geometry>
                 <box size="0.0225 0.2 0.05"/>
             </geometry>
-            <material name="orange"/>
+            <material name="black"/>
         </visual>
         <collision>
-            <origin xyz="0.075 -0.10 0.05" rpy="0 0 0"/>
+            <origin xyz="0.025 -0.10 0.025" rpy="0 0 0"/>
             <geometry>
                 <box size="0.0225 0.2 0.1"/>
@@ -109,5 +109,5 @@
         </collision>
         <xacro:inertial_box mass="0.3" x="0.0225" y="0.2" z="0.05" >
-            <origin xyz="0.075 -0.10 0.05" rpy="0 0 0"/>
+            <origin xyz="0.025 -0.10 0.025" rpy="0 0 0"/>
         </xacro:inertial_box>
     </link>
@@ -140,5 +140,5 @@
     <!-- Gazebo Simulation for Gripper -->
     <gazebo reference="gripper_base">
-        <material>Gazebo/Gray</material>
+        <material>Gazebo/Gold</material>
         <gravity>true</gravity>
         <ode>
@@ -148,5 +148,5 @@
     </gazebo>
     <gazebo reference="gripper_finger_left">
-        <material>Gazebo/Orange</material>
+        <material>Gazebo/Black</material>
         <gravity>true</gravity>
         <ode>
@@ -160,5 +160,5 @@
     </gazebo>
     <gazebo reference="gripper_finger_right">
-        <material>Gazebo/Orange</material>
+        <material>Gazebo/Black</material>
         <gravity>true</gravity>
         <ode>

File: src/articubot_one/description/robot_core.xacro (robot description, xacro)
@@ -4,24 +4,9 @@
         <color rgba="1 1 1 1" />
     </material>
-    <material name="orange">
-        <color rgba="1 0.3 0.1 1"/>
-    </material>
-    <material name="blue">
-        <color rgba="0.2 0.2 1 1"/>
-    </material>
     <material name="black">
         <color rgba="0 0 0 1"/>
     </material>
-    <material name="red">
-        <color rgba="1 0 0 1"/>
-    </material>
-    <material name="green">
-        <color rgba="0 1 0 1" />
-    </material>
     <material name="gray">
         <color rgba="0.5 0.5 0.5 1" />
-    </material>
-    <material name="pink">
-        <color rgba="1 0.4 0.7 1" />
     </material>
     <!-- BASE LINK -->
@@ -50,5 +35,5 @@
                 <cylinder length="0.15" radius="0.075"/>
             </geometry>
-            <material name="white"/>
+            <material name="gray"/>
         </visual>
         <collision>
@@ -60,10 +45,10 @@
             </geometry>
         </collision>
-        <xacro:inertial_box mass="200" x="0.451" y="0.451" z="0.18">
+        <xacro:inertial_box mass="500" x="0.451" y="0.451" z="0.18">
             <origin xyz="0 0 0.13" rpy="0 0 0"/>
         </xacro:inertial_box>
     </link>
     <gazebo reference="chassis">
-        <material>Gazebo/White</material>
+        <material>Gazebo/BuildingFrame</material>
     </gazebo>
     <!-- Wheel Link -->
@@ -73,5 +58,5 @@
                 <cylinder length="0.03" radius="0.07" />
             </geometry>
-            <material name="blue"/>
+            <material name="black"/>
         </visual>
         <collision>
@@ -85,5 +70,5 @@
     </link>
     <gazebo reference="front_left_wheel">
-        <material>Gazebo/Blue</material>
+        <material>Gazebo/GreyGradientSky</material>
     </gazebo>
     <link name="front_right_wheel">
@@ -92,5 +77,5 @@
                 <cylinder length="0.03" radius="0.07" />
             </geometry>
-            <material name="red"/>
+            <material name="black"/>
         </visual>
         <collision>
@@ -104,5 +89,5 @@
     </link>
     <gazebo reference="front_right_wheel">
-        <material>Gazebo/Red</material>
+        <material>Gazebo/GreyGradientSky</material>
     </gazebo>
     <link name="back_left_wheel">
@@ -111,5 +96,5 @@
                 <cylinder length="0.03" radius="0.07" />
             </geometry>
-            <material name="orange"/>
+            <material name="black"/>
         </visual>
         <collision>
@@ -123,5 +108,5 @@
     </link>
     <gazebo reference="back_left_wheel">
-        <material>Gazebo/Orange</material>
+        <material>Gazebo/GreyGradientSky</material>
     </gazebo>
     <link name="back_right_wheel">
@@ -130,5 +115,5 @@
                 <cylinder length="0.03" radius="0.07" />
             </geometry>
-            <material name="green"/>
+            <material name="black"/>
         </visual>
         <collision>
@@ -142,5 +127,5 @@
     </link>
     <gazebo reference="back_right_wheel">
-        <material>Gazebo/Green</material>
+        <material>Gazebo/GreyGradientSky</material>
     </gazebo>
     <!-- Wheel Joint -->
